Commit message: gazeboシミュレータで走行可否判定アルゴリズムを検証できるようにした

File: seniorcar_gazebo_simulator/urdf/base.urdf.xacro (robot description, xacro)
@@ -37,10 +37,10 @@
   <property name="chassis_width" value="0.711" />
   <property name="chassis_height" value="0.495" />
-  <property name="chassis_mass" value="487" />
-  <property name="front_axle_mass" value="113" />
+  <property name="chassis_mass" value="20" />
+  <property name="front_axle_mass" value="15" />
   <property name="front_axle_radius" value="0.13" />
   <property name="front_axle_length" value="1.0" />
-  <property name="base_x_origin_to_wheel_origin" value="0.448" /> <!-- 240/2 + 660/2-->
-  <property name="base_y_origin_to_wheel_origin" value="0.499" /> <!--(1282-711)/4 + 711/2-->
+  <property name="base_x_origin_to_wheel_origin" value="0.948" /> <!-- 240/2 + 660/2 changed from 0.448-->
+  <property name="base_y_origin_to_wheel_origin" value="0.499" /> <!--(1282-711)/4 + 711/2 = 1282/4 + 711/2 -->
   <property name="base_z_origin_to_wheel_origin" value="0.0" />
   <!-- Root link of Grizzly -->
@@ -139,15 +139,9 @@
   </link>
   <joint name="front_axle_joint"
-         type="revolute">
+         type="fixed">
     <origin xyz="${base_x_origin_to_wheel_origin} 0 0"
             rpy="0 0 0" />
     <parent link="chassis_link" />
     <child link="front_axle_link" />
-    <axis xyz="1 0 0"
-          rpy="0 0 0" />
-    <limit effort="10"
-           lower="-0.2"
-           upper="0.2"
-           velocity="0.5" />
   </joint>
   <grizzly_wheel fr="front" lr="left" parent="front_axle_link"
@@ -201,5 +195,5 @@
   <joint name="hokuyo_joint" type="fixed">
     <axis xyz="0 0 0" />
-    <origin xyz="0.0 0.0 0.1" rpy="0 0 0"/>
+    <origin xyz="0.0 0.0 0.3" rpy="0 0.5 0"/>
     <parent link="pico_flexx_link_optical_frame"/>
     <child link="hokuyo_link"/>
@@ -207,5 +201,5 @@
   <link name="hokuyo_link">
     <collision>
-      <origin xyz="0 0 0" rpy="0 0 0"/>
+      <origin xyz="0 0 0" rpy="0 0.5 0"/>
       <geometry>
         <box size="0.01 0.01 0.01"/>
@@ -251,3 +245,29 @@
     </inertial>
   </link>
+  <!-- human wieght -->
+  <joint name="human_mass_joint" type="fixed">
+    <axis xyz="0 0 0" />
+    <origin xyz="0.0 0.0 2.0" rpy="0 0 0"/>
+    <parent link="base_link"/>
+    <child link="human_mass_link"/>
+  </joint>
+  <link name="human_mass_link">
+    <collision>
+      <origin xyz="0 0 0" rpy="0 0 0"/>
+      <geometry>
+        <box size="0.1 0.1 0.1"/>
+      </geometry>
+    </collision>
+    <visual>
+      <origin xyz="0 0 0" rpy="0 0 0"/>
+      <geometry>
+        <box size="1 1 1"/>
+      </geometry>
+    </visual>
+    <inertial>
+      <mass value="50" />
+      <origin xyz="0 -0.3 0" rpy="0 0 0"/>
+      <inertia ixx="10" ixy="0" ixz="0" iyy="10" iyz="0" izz="10" />
+    </inertial>
+  </link>
 </robot>

File: seniorcar_gazebo_simulator/urdf/wheel.urdf.xacro (robot description, xacro)
@@ -27,7 +27,7 @@
 -->
 <robot name="grizzly_wheel" xmlns:xacro="http://ros.org/wiki/xacro">
-  <property name="wheel_mass" value="15" />
+  <property name="wheel_mass" value="1" />
   <property name="wheel_radius" value="0.33" />
-  <property name="wheel_width" value="0.252" />
+  <property name="wheel_width" value="0.1" />
   <xacro:macro name="grizzly_wheel"
                params="fr lr parent translateX translateY flipY">
@@ -58,7 +58,7 @@
     </link>
     <gazebo reference="${fr}_${lr}_wheel">
-      <mu1 value="1.0" />
-      <mu2 value="1.0" />
-      <kp value="10000000.0" />
+      <mu1 value="0.7" />
+      <mu2 value="0.7" />
+      <kp value="1000000.0" />
       <kd value="1.0" />
       <fdir1 value="1 0 0" />

Commit message: 透過率計算用ボクセルマップ作成 事故予見からの操舵回避デモ用プログラム作成 オドメトリ計算のバグを修正

File: seniorcar_gazebo_simulator/urdf/base.urdf.xacro (robot description, xacro)
@@ -37,10 +37,10 @@
   <property name="chassis_width" value="0.711" />
   <property name="chassis_height" value="0.495" />
-  <property name="chassis_mass" value="20" />
-  <property name="front_axle_mass" value="15" />
+  <property name="chassis_mass" value="487" />
+  <property name="front_axle_mass" value="113" />
   <property name="front_axle_radius" value="0.13" />
   <property name="front_axle_length" value="1.0" />
-  <property name="base_x_origin_to_wheel_origin" value="0.948" /> <!-- 240/2 + 660/2 changed from 0.448-->
-  <property name="base_y_origin_to_wheel_origin" value="0.499" /> <!--(1282-711)/4 + 711/2 = 1282/4 + 711/2 -->
+  <property name="base_x_origin_to_wheel_origin" value="0.448" /> <!-- 240/2 + 660/2-->
+  <property name="base_y_origin_to_wheel_origin" value="0.499" /> <!--(1282-711)/4 + 711/2-->
   <property name="base_z_origin_to_wheel_origin" value="0.0" />
   <!-- Root link of Grizzly -->
@@ -195,5 +195,5 @@
   <joint name="hokuyo_joint" type="fixed">
     <axis xyz="0 0 0" />
-    <origin xyz="0.0 0.0 0.3" rpy="0 0.5 0"/>
+    <origin xyz="0.0 0.0 0.8" rpy="0 0.4 0"/>
     <parent link="pico_flexx_link_optical_frame"/>
     <child link="hokuyo_link"/>
@@ -201,5 +201,5 @@
   <link name="hokuyo_link">
     <collision>
-      <origin xyz="0 0 0" rpy="0 0.5 0"/>
+      <origin xyz="0 0 0" rpy="0 0.4 0"/>
       <geometry>
         <box size="0.01 0.01 0.01"/>
@@ -246,4 +246,5 @@
   </link>
   <!-- human wieght -->
+  <!--
   <joint name="human_mass_joint" type="fixed">
     <axis xyz="0 0 0" />
@@ -271,3 +272,4 @@
     </inertial>
   </link>
+-->
 </robot>

File: seniorcar_gazebo_simulator/urdf/wheel.urdf.xacro (robot description, xacro)
@@ -27,5 +27,5 @@
 -->
 <robot name="grizzly_wheel" xmlns:xacro="http://ros.org/wiki/xacro">
-  <property name="wheel_mass" value="1" />
+  <property name="wheel_mass" value="10" />
   <property name="wheel_radius" value="0.33" />
   <property name="wheel_width" value="0.1" />
